File: pcb/kicad/fpga.sch (KiCad schematic (older format))
At the start: 16 parts, among them P3 CONN_2, U4 XC3S400-PQ208

Commit message: pcb wip
Parts:
- added C38, C39: 100n, symbol C
Connections:
- net +1.2V: now also C38.1, C39.1
- net GND: now also C38.2, C39.2
