File: pcb/kicad/fpga.sch (KiCad schematic (older format))
At the start: 18 parts, among them P3 CONN_2, U4 XC3S400-PQ208

Commit message: pcb+schem wip
Other:
- note added: "55ns SRAM bus"
- note added: "70ns PSRAM bus"
- note added: "DAC"
- note added: "FPGA"
- note added: "Freeze button"
- note added: "SNES A+B bus"
- note added: "SPI (MCU)"
- note added: "SPI (SD); shared with MCU"
Changed lines of the file:
@@
-EESchema Schematic File Version 2  date Wed 02 Jun 2010 02:08:21 PM CEST
+EESchema Schematic File Version 2  date Fri 04 Jun 2010 01:55:30 AM CEST
 LIBS:power
 LIBS:device
@@
 Sheet 6 6
 Title "sd2snes Mark II"
-Date "2 jun 2010"
+Date "3 jun 2010"
 Rev "A"
 Comp "Maximilian Rehkopf"
@@
 Comment4 ""
 $EndDescr
+Text Notes 11850 10450 0    500  ~ 100
+FPGA
+Text Notes 12800 8150 1    50   ~ 0
+SNES A+B bus
+Text Notes 11800 4500 1    50   ~ 0
+70ns PSRAM bus
+Text Notes 4650 5600 1    50   ~ 0
+55ns SRAM bus
+Text Notes 2800 7400 0    50   ~ 0
+SPI (SD); shared with MCU
+Text Notes 3450 7800 0    50   ~ 0
+SPI (MCU)
+Text Notes 3700 8150 0    50   ~ 0
+DAC
+Text Notes 1250 7000 0    50   ~ 0
+Freeze button
 Connection ~ 4850 10950
 Wire Wire Line

Commit message: pcb wip
Parts:
- added P79: CONN_1, symbol CONN_1
- C18, C19, C20, C21, C22, C23, C24, C25, C26, C27, C28, C29, C30, C31, C38, C39: footprint (none) -> SM0805_FIXEDMASK
- P3: footprint (none) -> PIN_ARRAY_2X1
- U4: footprint (none) -> PQFP208
Connections:
- net at U4.79 (IO_L32P_4/GCLK0): now also P79.1
