File: pcb/kicad/snesslot.sch (KiCad schematic (older format))
At the start: 18 parts, among them J1 SNESCART_EXT, U1 74ALVC164245, U2 74ALVC164245, U3 74ALVC164245, U5 74LVC1T45

Commit message: pcb+schem wip
Other:
- note added: "SNES bus,\nlevel shift"
Changed lines of the file:
@@
-EESchema Schematic File Version 2  date Wed 02 Jun 2010 02:08:21 PM CEST
+EESchema Schematic File Version 2  date Fri 04 Jun 2010 01:55:30 AM CEST
 LIBS:power
 LIBS:device
@@
 Sheet 2 6
 Title "sd2snes Mark II"
-Date "2 jun 2010"
+Date "3 jun 2010"
 Rev "A"
 Comp "Maximilian Rehkopf"
@@
 Comment4 ""
 $EndDescr
+Text Notes 7100 6550 0    250  ~ 50
+SNES bus,\nlevel shift
 Wire Wire Line
 	6550 6850 6550 6700

Commit message: pcb wip
Parts:
- R1: value 300 -> 330
Changed lines of the file:
@@
-EESchema Schematic File Version 2  date Tue 08 Jun 2010 04:15:56 AM CEST
+EESchema Schematic File Version 2  date Thu 10 Jun 2010 11:56:43 PM CEST
 LIBS:power
 LIBS:device
@@
 Sheet 2 6
 Title "sd2snes Mark II"
-Date "8 jun 2010"
+Date "10 jun 2010"
 Rev "A"
 Comp "Maximilian Rehkopf"
@@
 P 4850 5650
 F 0 "R1" V 4930 5650 50  0000 C CNN
-F 1 "300" V 4850 5650 50  0000 C CNN
+F 1 "330" V 4850 5650 50  0000 C CNN
 	1    4850 5650
 	1    0    0    -1

Commit message: pcb wip
Parts:
- C10, C11, C12, C13, C14, C52, C53, C54, C55, C56, C57, C9, R1: footprint (none) -> SM0805_FIXEDMASK
- J1: footprint (none) -> SNESCART_EXT
- U1, U2, U3: footprint (none) -> TSSOP48
- U5: footprint (none) -> SOT563
Changed lines of the file:
@@
-EESchema Schematic File Version 2  date Thu 10 Jun 2010 11:56:43 PM CEST
+EESchema Schematic File Version 2  date Fri 11 Jun 2010 11:43:50 PM CEST
 LIBS:power
 LIBS:device
@@
 Sheet 2 6
 Title "sd2snes Mark II"
-Date "10 jun 2010"
+Date "11 jun 2010"
 Rev "A"
 Comp "Maximilian Rehkopf"
@@
 	6550 7250 6550 7400
 $Comp
-L GND #PWR19
+L GND #PWR01
 U 1 1 4BAD42F7
 P 5550 7500
-F 0 "#PWR19" H 5550 7500 30  0001 C CNN
+F 0 "#PWR01" H 5550 7500 30  0001 C CNN
 F 1 "GND" H 5550 7430 30  0001 C CNN
 	1    5550 7500
@@
 F 0 "C55" H 5600 7150 50  0000 L CNN
 F 1 "100n" H 5600 6950 50  0000 L CNN
+F 2 "SM0805_FIXEDMASK" H 5550 7050 60  0001 C CNN
 	1    5550 7050
 	1    0    0    -1
@@
 F 0 "C56" H 5850 7150 50  0000 L CNN
 F 1 "100n" H 5850 6950 50  0000 L CNN
+F 2 "SM0805_FIXEDMASK" H 5800 7050 60  0001 C CNN
 	1    5800 7050
 	1    0    0    -1
@@
 F 0 "C57" H 6100 7150 50  0000 L CNN
 F 1 "100n" H 6100 6950 50  0000 L CNN
+F 2 "SM0805_FIXEDMASK" H 6050 7050 60  0001 C CNN
 	1    6050 7050
 	1    0    0    -1
@@
 F 0 "C54" H 5250 7150 50  0000 L CNN
 F 1 "100n" H 5250 6950 50  0000 L CNN
+F 2 "SM0805_FIXEDMASK" H 5200 7050 60  0001 C CNN
 	1    5200 7050
 	1    0    0    -1
@@
 F 0 "C53" H 5000 7150 50  0000 L CNN
 F 1 "100n" H 5000 6950 50  0000 L CNN
+F 2 "SM0805_FIXEDMASK" H 4950 7050 60  0001 C CNN
 	1    4950 7050
 	1    0    0    -1
@@
 F 0 "C52" H 4750 7150 50  0000 L CNN
 F 1 "100n" H 4750 6950 50  0000 L CNN
+F 2 "SM0805_FIXEDMASK" H 4700 7050 60  0001 C CNN
 	1    4700 7050
 	1    0    0    -1
@@
 IRQ_DIR
 $Comp
-L GND #PWR13
+L GND #PWR02
 U 1 1 4BAEAB97
 P 3150 5950
-F 0 "#PWR13" H 3150 5950 30  0001 C CNN
+F 0 "#PWR02" H 3150 5950 30  0001 C CNN
 F 1 "GND" H 3150 5880 30  0001 C CNN
 	1    3150 5950
@@
 $EndComp
 $Comp
-L GND #PWR14
+L GND #PWR03
 U 1 1 4BAEAB8D
 P 3150 6950
-F 0 "#PWR14" H 3150 6950 30  0001 C CNN
+F 0 "#PWR03" H 3150 6950 30  0001 C CNN
 F 1 "GND" H 3150 6880 30  0001 C CNN
 	1    3150 6950
@@
 $EndComp
 $Comp
-L GND #PWR11
+L GND #PWR04
 U 1 1 4BAEAB85
 P 3150 2250
-F 0 "#PWR11" H 3150 2250 30  0001 C CNN
+F 0 "#PWR04" H 3150 2250 30  0001 C CNN
 F 1 "GND" H 3150 2180 30  0001 C CNN
 	1    3150 2250
@@
 $EndComp
 $Comp
-L GND #PWR12
+L GND #PWR05
 U 1 1 4BAEAB7E
 P 3150 3250
-F 0 "#PWR12" H 3150 3250 30  0001 C CNN
+F 0 "#PWR05" H 3150 3250 30  0001 C CNN
 F 1 "GND" H 3150 3180 30  0001 C CNN
 	1    3150 3250
@@
 $EndComp
 $Comp
-L GND #PWR22
+L GND #PWR06
 U 1 1 4BAEAB58
 P 8400 2250
-F 0 "#PWR22" H 8400 2250 30  0001 C CNN
+F 0 "#PWR06" H 8400 2250 30  0001 C CNN
 F 1 "GND" H 8400 2180 30  0001 C CNN
 	1    8400 2250
@@
 $EndComp
 $Comp
-L GND #PWR29
+L GND #PWR07
 U 1 1 4BAEAAFB
 P 10400 2250
-F 0 "#PWR29" H 10400 2250 30  0001 C CNN
+F 0 "#PWR07" H 10400 2250 30  0001 C CNN
 F 1 "GND" H 10400 2180 30  0001 C CNN
 	1    10400 2250
@@
 $EndComp
 $Comp
-L GND #PWR4
+L GND #PWR08
 U 1 1 4BAEAAF9
 P 1150 6950
-F 0 "#PWR4" H 1150 6950 30  0001 C CNN
+F 0 "#PWR08" H 1150 6950 30  0001 C CNN
 F 1 "GND" H 1150 6880 30  0001 C CNN
 	1    1150 6950
@@
 $EndComp
 $Comp
-L GND #PWR2
+L GND #PWR09
 U 1 1 4BAEAAF5
 P 1150 3250
-F 0 "#PWR2" H 1150 3250 30  0001 C CNN
+F 0 "#PWR09" H 1150 3250 30  0001 C CNN
 F 1 "GND" H 1150 3180 30  0001 C CNN
 	1    1150 3250
@@
 $EndComp
 $Comp
-L GND #PWR3
+L GND #PWR010
 U 1 1 4BAEAAEF
 P 1150 5950
-F 0 "#PWR3" H 1150 5950 30  0001 C CNN
+F 0 "#PWR010" H 1150 5950 30  0001 C CNN
 F 1 "GND" H 1150 5880 30  0001 C CNN
 	1    1150 5950
@@
 $EndComp
 $Comp
-L GND #PWR1
+L GND #PWR011
 U 1 1 4BAEAAE9
 P 1150 2250
-F 0 "#PWR1" H 1150 2250 30  0001 C CNN
+F 0 "#PWR011" H 1150 2250 30  0001 C CNN
 F 1 "GND" H 1150 2180 30  0001 C CNN
 	1    1150 2250
@@
 SNES_A15
 $Comp
-L GND #PWR17
+L GND #PWR012
 U 1 1 4BAE51D9
 P 4850 6000
-F 0 "#PWR17" H 4850 6000 30  0001 C CNN
+F 0 "#PWR012" H 4850 6000 30  0001 C CNN
 F 1 "GND" H 4850 5930 30  0001 C CNN
 	1    4850 6000
@@
 F 0 "R1" V 4930 5650 50  0000 C CNN
 F 1 "330" V 4850 5650 50  0000 C CNN
+F 2 "SM0805_FIXEDMASK" H 4850 5650 60  0001 C CNN
 	1    4850 5650
 	1    0    0    -1
@@
 SNES_EXT_A0
 $Comp
-L GND #PWR26
+L GND #PWR013
 U 1 1 4BAD4383
 P 9400 6300
-F 0 "#PWR26" H 9400 6300 30  0001 C CNN
+F 0 "#PWR013" H 9400 6300 30  0001 C CNN
 F 1 "GND" H 9400 6230 30  0001 C CNN
 	1    9400 6300
@@
 $EndComp
 $Comp
-L +3.3V #PWR27
+L +3.3V #PWR014
 U 1 1 4BAD437E
 P 9500 4650
-F 0 "#PWR27" H 9500 4610 30  0001 C CNN
+F 0 "#PWR014" H 9500 4610 30  0001 C CNN
 F 1 "+3.3V" H 9500 4760 30  0000 C CNN
 	1    9500 4650
@@
 $EndComp
 $Comp
-L +5V #PWR24
+L +5V #PWR015
 U 1 1 4BAD4372
 P 9300 4650
-F 0 "#PWR24" H 9300 4740 20  0001 C CNN
+F 0 "#PWR015" H 9300 4740 20  0001 C CNN
 F 1 "+5V" H 9300 4740 30  0000 C CNN
 	1    9300 4650
@@
 F 0 "C14" H 6850 7150 50  0000 L CNN
 F 1 "100n" H 6850 6950 50  0000 L CNN
+F 2 "SM0805_FIXEDMASK" H 6800 7050 60  0001 C CNN
 	1    6800 7050
 	1    0    0    -1
@@
 F 0 "C13" H 6600 7150 50  0000 L CNN
 F 1 "100n" H 6600 6950 50  0000 L CNN
+F 2 "SM0805_FIXEDMASK" H 6550 7050 60  0001 C CNN
 	1    6550 7050
 	1    0    0    -1
@@
 F 0 "C12" H 6350 7150 50  0000 L CNN
 F 1 "100n" H 6350 6950 50  0000 L CNN
+F 2 "SM0805_FIXEDMASK" H 6300 7050 60  0001 C CNN
 	1    6300 7050
 	1    0    0    -1
@@
 F 0 "C11" H 4500 7150 50  0000 L CNN
 F 1 "100n" H 4500 6950 50  0000 L CNN
+F 2 "SM0805_FIXEDMASK" H 4450 7050 60  0001 C CNN
 	1    4450 7050
 	1    0    0    -1
@@
 F 0 "C10" H 4250 7150 50  0000 L CNN
 F 1 "100n" H 4250 6950 50  0000 L CNN
+F 2 "SM0805_FIXEDMASK" H 4200 7050 60  0001 C CNN
 	1    4200 7050
 	1    0    0    -1
@@
 F 0 "C9" H 4000 7150 50  0000 L CNN
 F 1 "100n" H 4000 6950 50  0000 L CNN
+F 2 "SM0805_FIXEDMASK" H 3950 7050 60  0001 C CNN
 	1    3950 7050
 	1    0    0    -1
 $EndComp
 $Comp
-L GND #PWR16
+L GND #PWR016
 U 1 1 4BAD42C1
 P 3950 7500
-F 0 "#PWR16" H 3950 7500 30  0001 C CNN
+F 0 "#PWR016" H 3950 7500 30  0001 C CNN
 F 1 "GND" H 3950 7430 30  0001 C CNN
 	1    3950 7500
@@
 $EndComp
 $Comp
-L +5V #PWR18
+L +5V #PWR017
 U 1 1 4BAD42B7
 P 5550 6600
-F 0 "#PWR18" H 5550 6690 20  0001 C CNN
+F 0 "#PWR017" H 5550 6690 20  0001 C CNN
 F 1 "+5V" H 5550 6690 30  0000 C CNN
 	1    5550 6600
@@
 $EndComp
 $Comp
-L +3.3V #PWR15
+L +3.3V #PWR018
 U 1 1 4BAD42B3
 P 3950 6600
-F 0 "#PWR15" H 3950 6560 30  0001 C CNN
+F 0 "#PWR018" H 3950 6560 30  0001 C CNN
 F 1 "+3.3V" H 3950 6710 30  0000 C CNN
 	1    3950 6600
@@
 $EndComp
 $Comp
-L +3.3V #PWR5
+L +3.3V #PWR019
 U 1 1 4B6ED29E
 P 2000 600
-F 0 "#PWR5" H 2000 560 30  0001 C CNN
+F 0 "#PWR019" H 2000 560 30  0001 C CNN
 F 1 "+3.3V" H 2000 710 30  0000 C CNN
 	1    2000 600
@@
 $EndComp
 $Comp
-L +3.3V #PWR6
+L +3.3V #PWR020
 U 1 1 4B6ED291
 P 2000 4300
-F 0 "#PWR6" H 2000 4260 30  0001 C CNN
+F 0 "#PWR020" H 2000 4260 30  0001 C CNN
 F 1 "+3.3V" H 2000 4410 30  0000 C CNN
 	1    2000 4300
@@
 F 0 "U5" H 9400 5450 60  0000 C CNN
 F 1 "74LVC1T45" H 9650 5050 60  0000 C CNN
+F 2 "SOT563" H 9400 5450 60  0001 C CNN
 	1    9400 5450
 	-1   0    0    -1
 $EndComp
 $Comp
-L +3.3V #PWR28
+L +3.3V #PWR021
 U 1 1 4B6E9E3A
 P 9550 600
-F 0 "#PWR28" H 9550 560 50  0001 C CNN
+F 0 "#PWR021" H 9550 560 50  0001 C CNN
 F 1 "+3.3V" H 9400 650 50  0000 C CNN
 	1    9550 600
@@
 $EndComp
 $Comp
-L +5V #PWR10
+L +5V #PWR022
 U 1 1 4B6E9DCF
 P 2300 4300
-F 0 "#PWR10" H 2300 4390 20  0001 C CNN
+F 0 "#PWR022" H 2300 4390 20  0001 C CNN
 F 1 "+5V" H 2300 4390 30  0000 C CNN
 	1    2300 4300
@@
 $EndComp
 $Comp
-L +5V #PWR9
+L +5V #PWR023
 U 1 1 4B6E9DCB
 P 2300 600
-F 0 "#PWR9" H 2300 690 20  0001 C CNN
+F 0 "#PWR023" H 2300 690 20  0001 C CNN
 F 1 "+5V" H 2300 690 30  0000 C CNN
 	1    2300 600
@@
 $EndComp
 $Comp
-L +5V #PWR23
+L +5V #PWR024
 U 1 1 4B6E9DC6
 P 9250 600
-F 0 "#PWR23" H 9250 690 50  0001 C CNN
+F 0 "#PWR024" H 9250 690 50  0001 C CNN
 F 1 "+5V" H 9150 650 50  0000 C CNN
 	1    9250 600
@@
 $EndComp
 $Comp
-L +5V #PWR20
+L +5V #PWR025
 U 1 1 4B6E9D3D
 P 6050 1300
-F 0 "#PWR20" H 6050 1390 20  0001 C CNN
+F 0 "#PWR025" H 6050 1390 20  0001 C CNN
 F 1 "+5V" H 6050 1390 30  0000 C CNN
 	1    6050 1300
@@
 $EndComp
 $Comp
-L GND #PWR25
+L GND #PWR026
 U 1 1 4B6E9C12
 P 9400 4000
-F 0 "#PWR25" H 9400 4000 30  0001 C CNN
+F 0 "#PWR026" H 9400 4000 30  0001 C CNN
 F 1 "GND" H 9400 3930 30  0001 C CNN
 	1    9400 4000
@@
 $EndComp
 $Comp
-L GND #PWR7
+L GND #PWR027
 U 1 1 4B6E9C04
 P 2150 4000
-F 0 "#PWR7" H 2150 4000 30  0001 C CNN
+F 0 "#PWR027" H 2150 4000 30  0001 C CNN
 F 1 "GND" H 2150 3930 30  0001 C CNN
 	1    2150 4000
@@
 $EndComp
 $Comp
-L GND #PWR21
+L GND #PWR028
 U 1 1 4B6E9BA6
 P 6050 6000
-F 0 "#PWR21" H 6050 6000 30  0001 C CNN
+F 0 "#PWR028" H 6050 6000 30  0001 C CNN
 F 1 "GND" H 6050 5930 30  0001 C CNN
 	1    6050 6000
@@
 $EndComp
 $Comp
-L GND #PWR8
+L GND #PWR029
 U 1 1 4B6E9B44
 P 2150 7700
-F 0 "#PWR8" H 2150 7700 30  0001 C CNN
+F 0 "#PWR029" H 2150 7700 30  0001 C CNN
 F 1 "GND" H 2150 7630 30  0001 C CNN
 	1    2150 7700
@@
 F 0 "J1" H 5600 5500 60  0000 C CNN
 F 1 "SNESCART_EXT" H 6550 1600 60  0000 C CNN
+F 2 "SNESCART_EXT" H 6050 3600 60  0001 C CNN
 	1    6050 3600
 	1    0    0    -1
@@
 F 0 "U3" H 2150 2400 60  0000 C CNN
 F 1 "74ALVC164245" H 2150 2300 60  0000 C CNN
+F 2 "TSSOP48" H 2150 2300 60  0001 C CNN
 	1    2150 2300
 	1    0    0    -1
@@
 F 0 "U2" H 2150 6100 60  0000 C CNN
 F 1 "74ALVC164245" H 2150 6000 60  0000 C CNN
+F 2 "TSSOP48" H 2150 6000 60  0001 C CNN
 	1    2150 6000
 	1    0    0    -1
@@
 F 0 "U1" H 9400 2400 60  0000 C CNN
 F 1 "74ALVC164245" H 9400 2300 60  0000 C CNN
+F 2 "TSSOP48" H 9400 2300 60  0001 C CNN
 	1    9400 2300
 	-1   0    0    -1
