File: pcb/kicad/snesslot.sch (KiCad schematic (older format))
At the start: 18 parts, among them J1 SNESCART_EXT, U1 74ALVC164245, U2 74ALVC164245, U3 74ALVC164245, U5 74LVC1T45

Commit message: pcb wip (cleanup silk screen)
Connections:
- no-connect marks 0 -> 2
Changed lines of the file:
@@
-EESchema Schematic File Version 2  date Mon 02 Aug 2010 11:18:19 PM CEST
+EESchema Schematic File Version 2  date Tue 03 Aug 2010 15:22:28 CEST
 LIBS:power
 LIBS:device
@@
 Sheet 2 6
 Title "sd2snes Mark II"
-Date "2 aug 2010"
+Date "3 aug 2010"
 Rev "A"
 Comp "Maximilian Rehkopf"
@@
 Comment4 ""
 $EndDescr
-Text Notes 7100 6550 0    250  ~ 50
-SNES bus,\nlevel shift
+NoConn ~ 7050 4200
+NoConn ~ 7050 4400
+Wire Wire Line
+	6850 4400 7050 4400
 Wire Wire Line
 	6550 6850 6550 6700
@@
 Wire Wire Line
 	6550 7250 6550 7400
+Wire Wire Line
+	6850 4200 7050 4200
+Text Notes 7100 6550 0    250  ~ 50
+SNES bus,\nlevel shift
 $Comp
 L GND #PWR01

Commit message: pcb wip (relabel components)
Parts:
- renumbered C9 to C101, C10 to C102, C11 to C103, C52 to C104, C53 to C105, C54 to C106, C55 to C111, C56 to C112, C57 to C113, C12 to C114, C13 to C115, C14 to C116, J1 to J101, R1 to R101, U1 to U101, U2 to U102, U3 to U103, U5 to U104
Changed lines of the file:
@@
-EESchema Schematic File Version 2  date Tue 03 Aug 2010 15:22:28 CEST
+EESchema Schematic File Version 2  date Wed 04 Aug 2010 09:24:14 CEST
 LIBS:power
 LIBS:device
@@
 Sheet 2 6
 Title "sd2snes Mark II"
-Date "3 aug 2010"
+Date "4 aug 2010"
 Rev "A"
 Comp "Maximilian Rehkopf"
@@
 $EndComp
 $Comp
-L C C55
+L C C111
 U 1 1 4BFB119A
 P 5550 7050
-F 0 "C55" H 5600 7150 50  0000 L CNN
+F 0 "C111" H 5600 7150 50  0000 L CNN
 F 1 "100n" H 5600 6950 50  0000 L CNN
 F 2 "SM0805_FIXEDMASK" H 5550 7050 60  0001 C CNN
@@
 $EndComp
 $Comp
-L C C56
+L C C112
 U 1 1 4BFB1199
 P 5800 7050
-F 0 "C56" H 5850 7150 50  0000 L CNN
+F 0 "C112" H 5850 7150 50  0000 L CNN
 F 1 "100n" H 5850 6950 50  0000 L CNN
 F 2 "SM0805_FIXEDMASK" H 5800 7050 60  0001 C CNN
@@
 $EndComp
 $Comp
-L C C57
+L C C113
 U 1 1 4BFB1197
 P 6050 7050
-F 0 "C57" H 6100 7150 50  0000 L CNN
+F 0 "C113" H 6100 7150 50  0000 L CNN
 F 1 "100n" H 6100 6950 50  0000 L CNN
 F 2 "SM0805_FIXEDMASK" H 6050 7050 60  0001 C CNN
@@
 $EndComp
 $Comp
-L C C54
+L C C106
 U 1 1 4BFB1194
 P 5200 7050
-F 0 "C54" H 5250 7150 50  0000 L CNN
+F 0 "C106" H 5250 7150 50  0000 L CNN
 F 1 "100n" H 5250 6950 50  0000 L CNN
 F 2 "SM0805_FIXEDMASK" H 5200 7050 60  0001 C CNN
@@
 $EndComp
 $Comp
-L C C53
+L C C105
 U 1 1 4BFB1192
 P 4950 7050
-F 0 "C53" H 5000 7150 50  0000 L CNN
+F 0 "C105" H 5000 7150 50  0000 L CNN
 F 1 "100n" H 5000 6950 50  0000 L CNN
 F 2 "SM0805_FIXEDMASK" H 4950 7050 60  0001 C CNN
@@
 $EndComp
 $Comp
-L C C52
+L C C104
 U 1 1 4BFB1190
 P 4700 7050
-F 0 "C52" H 4750 7150 50  0000 L CNN
+F 0 "C104" H 4750 7150 50  0000 L CNN
 F 1 "100n" H 4750 6950 50  0000 L CNN
 F 2 "SM0805_FIXEDMASK" H 4700 7050 60  0001 C CNN
@@
 $EndComp
 $Comp
-L R R1
+L R R101
 U 1 1 4BAE51CA
 P 4850 5650
-F 0 "R1" V 4930 5650 50  0000 C CNN
+F 0 "R101" V 4930 5650 50  0000 C CNN
 F 1 "220" V 4850 5650 50  0000 C CNN
 F 2 "SM0805_FIXEDMASK" H 4850 5650 60  0001 C CNN
@@
 $EndComp
 $Comp
-L C C14
+L C C116
 U 1 1 4BAD42E2
 P 6800 7050
-F 0 "C14" H 6850 7150 50  0000 L CNN
+F 0 "C116" H 6850 7150 50  0000 L CNN
 F 1 "100n" H 6850 6950 50  0000 L CNN
 F 2 "SM0805_FIXEDMASK" H 6800 7050 60  0001 C CNN
@@
 $EndComp
 $Comp
-L C C13
+L C C115
 U 1 1 4BAD42E0
 P 6550 7050
-F 0 "C13" H 6600 7150 50  0000 L CNN
+F 0 "C115" H 6600 7150 50  0000 L CNN
 F 1 "100n" H 6600 6950 50  0000 L CNN
 F 2 "SM0805_FIXEDMASK" H 6550 7050 60  0001 C CNN
@@
 $EndComp
 $Comp
-L C C12
+L C C114
 U 1 1 4BAD42DF
 P 6300 7050
-F 0 "C12" H 6350 7150 50  0000 L CNN
+F 0 "C114" H 6350 7150 50  0000 L CNN
 F 1 "100n" H 6350 6950 50  0000 L CNN
 F 2 "SM0805_FIXEDMASK" H 6300 7050 60  0001 C CNN
@@
 $EndComp
 $Comp
-L C C11
+L C C103
 U 1 1 4BAD42DA
 P 4450 7050
-F 0 "C11" H 4500 7150 50  0000 L CNN
+F 0 "C103" H 4500 7150 50  0000 L CNN
 F 1 "100n" H 4500 6950 50  0000 L CNN
 F 2 "SM0805_FIXEDMASK" H 4450 7050 60  0001 C CNN
@@
 $EndComp
 $Comp
-L C C10
+L C C102
 U 1 1 4BAD42D8
 P 4200 7050
-F 0 "C10" H 4250 7150 50  0000 L CNN
+F 0 "C102" H 4250 7150 50  0000 L CNN
 F 1 "100n" H 4250 6950 50  0000 L CNN
 F 2 "SM0805_FIXEDMASK" H 4200 7050 60  0001 C CNN
@@
 $EndComp
 $Comp
-L C C9
+L C C101
 U 1 1 4BAD42D5
 P 3950 7050
-F 0 "C9" H 4000 7150 50  0000 L CNN
+F 0 "C101" H 4000 7150 50  0000 L CNN
 F 1 "100n" H 4000 6950 50  0000 L CNN
 F 2 "SM0805_FIXEDMASK" H 3950 7050 60  0001 C CNN
@@
 $EndComp
 $Comp
-L 74LVC1T45 U5
+L 74LVC1T45 U104
 U 1 1 4B6EB593
 P 9400 5450
-F 0 "U5" H 9400 5450 60  0000 C CNN
+F 0 "U104" H 9400 5450 60  0000 C CNN
 F 1 "74LVC1T45" H 9650 5050 60  0000 C CNN
 F 2 "SOT563" H 9400 5450 60  0001 C CNN
@@
 $EndComp
 $Comp
-L SNESCART_EXT J1
+L SNESCART_EXT J101
 U 1 1 4B6E1766
 P 6050 3600
-F 0 "J1" H 5600 5500 60  0000 C CNN
+F 0 "J101" H 5600 5500 60  0000 C CNN
 F 1 "SNESCART_EXT" H 6550 1600 60  0000 C CNN
 F 2 "SNESCART_EXT" H 6050 3600 60  0001 C CNN
@@
 $EndComp
 $Comp
-L 74ALVC164245 U3
+L 74ALVC164245 U103
 U 1 1 4B6E1748
 P 2150 2300
-F 0 "U3" H 2150 2400 60  0000 C CNN
+F 0 "U103" H 2150 2400 60  0000 C CNN
 F 1 "74ALVC164245" H 2150 2300 60  0000 C CNN
 F 2 "TSSOP48" H 2150 2300 60  0001 C CNN
@@
 $EndComp
 $Comp
-L 74ALVC164245 U2
+L 74ALVC164245 U102
 U 1 1 4B6E1744
 P 2150 6000
-F 0 "U2" H 2150 6100 60  0000 C CNN
+F 0 "U102" H 2150 6100 60  0000 C CNN
 F 1 "74ALVC164245" H 2150 6000 60  0000 C CNN
 F 2 "TSSOP48" H 2150 6000 60  0001 C CNN
@@
 $EndComp
 $Comp
-L 74ALVC164245 U1
+L 74ALVC164245 U101
 U 1 1 4B6E1740
 P 9400 2300
-F 0 "U1" H 9400 2400 60  0000 C CNN
+F 0 "U101" H 9400 2400 60  0000 C CNN
 F 1 "74ALVC164245" H 9400 2300 60  0000 C CNN
 F 2 "TSSOP48" H 9400 2300 60  0001 C CNN
