File: pcb/kicad/mcu.sch (KiCad schematic (older format))
At the start: 11 parts, among them J2 SD_CARD, J3 USB_MINIB, P1 CONN_14, P2 CONN_2, U11 LPC1754, X1 12MHz, X2 32.768kHz

Commit message: pcb wip
Parts:
- added C40, C41, C42, C43, C44: C, symbol C
Connections:
- net +3.3V: now also C40.1, C41.1, C42.1, C43.1, C44.1
- net GND: now also C40.2, C41.2, C42.2, C43.2, C44.2
Changed lines of the file:
@@
-EESchema Schematic File Version 2  date Fri 21 May 2010 12:12:26 AM CEST
+EESchema Schematic File Version 2  date Fri 21 May 2010 07:28:17 PM CEST
 LIBS:power
 LIBS:device
@@
 Sheet 4 6
 Title "sd2snes Mark II"
-Date "20 may 2010"
+Date "21 may 2010"
 Rev "A"
 Comp "Maximilian Rehkopf"
@@
 Comment4 ""
 $EndDescr
-Text GLabel 2500 4800 0    50   Input ~ 0
-/TRST
+Connection ~ 8100 6850
+Wire Wire Line
+	8350 6750 8350 6850
+Wire Wire Line
+	8350 6850 7600 6850
+Connection ~ 7600 6850
+Wire Wire Line
+	7850 6850 7850 6750
+Connection ~ 7850 6250
+Wire Wire Line
+	8100 6250 8100 6350
+Wire Wire Line
+	7600 6350 7600 6150
 Wire Wire Line
 	3000 4800 2500 4800
@@
 Wire Wire Line
 	6500 2900 8850 2900
-Connection ~ 10200 3500
-Wire Wire Line
-	10200 3500 10100 3500
-Connection ~ 10200 3600
-Wire Wire Line
-	10200 3900 10200 3300
-Wire Wire Line
-	10200 3300 10100 3300
-Wire Wire Line
-	10200 2650 10200 2900
-Wire Wire Line
-	10200 2900 10100 2900
+Connection ~ 10400 3500
+Wire Wire Line
+	10400 3500 10100 3500
+Connection ~ 10400 3600
+Wire Wire Line
+	10400 3900 10400 3300
+Wire Wire Line
+	10400 3300 10100 3300
+Wire Wire Line
+	10400 2650 10400 2900
+Wire Wire Line
+	10400 2900 10100 2900
 Wire Wire Line
 	4250 6650 4250 6850
@@
 	4450 1450 4450 1550
 Wire Wire Line
-	10200 3600 10100 3600
-Wire Wire Line
-	10100 3400 10200 3400
-Connection ~ 10200 3400
+	10400 3600 10100 3600
+Wire Wire Line
+	10100 3400 10400 3400
+Connection ~ 10400 3400
 Wire Wire Line
 	7550 2800 6500 2800
@@
 Wire Wire Line
 	6500 2700 6800 2700
+Wire Wire Line
+	7600 6750 7600 6950
+Wire Wire Line
+	7850 6250 7850 6350
+Connection ~ 7600 6250
+Wire Wire Line
+	7600 6250 8350 6250
+Wire Wire Line
+	8350 6250 8350 6350
+Connection ~ 8100 6250
+Wire Wire Line
+	8100 6850 8100 6750
+Connection ~ 7850 6850
+$Comp
+L GND #PWR044
+U 1 1 4BF6C1FC
+P 7600 6950
+F 0 "#PWR044" H 7600 6950 30  0001 C CNN
+F 1 "GND" H 7600 6880 30  0001 C CNN
+	1    7600 6950
+	1    0    0    -1
+$EndComp
+$Comp
+L +3.3V #PWR045
+U 1 1 4BF6C1F7
+P 7600 6150
+F 0 "#PWR045" H 7600 6110 30  0001 C CNN
+F 1 "+3.3V" H 7600 6260 30  0000 C CNN
+	1    7600 6150
+	-1   0    0    -1
+$EndComp
+$Comp
+L C C43
+U 1 1 4BF6BFE6
+P 8350 6550
+F 0 "C43" H 8400 6650 50  0000 L CNN
+F 1 "C" H 8400 6450 50  0000 L CNN
+	1    8350 6550
+	1    0    0    -1
+$EndComp
+$Comp
+L C C42
+U 1 1 4BF6BFE5
+P 8100 6550
+F 0 "C42" H 8150 6650 50  0000 L CNN
+F 1 "C" H 8150 6450 50  0000 L CNN
+	1    8100 6550
+	1    0    0    -1
+$EndComp
+$Comp
+L C C41
+U 1 1 4BF6BFE2
+P 7850 6550
+F 0 "C41" H 7900 6650 50  0000 L CNN
+F 1 "C" H 7900 6450 50  0000 L CNN
+	1    7850 6550
+	1    0    0    -1
+$EndComp
+$Comp
+L C C40
+U 1 1 4BF6BFE1
+P 7600 6550
+F 0 "C40" H 7650 6650 50  0000 L CNN
+F 1 "C" H 7650 6450 50  0000 L CNN
+	1    7600 6550
+	1    0    0    -1
+$EndComp
+$Comp
+L C C44
+U 1 1 4BF6BFBB
+P 10400 3100
+F 0 "C44" H 10450 3200 50  0000 L CNN
+F 1 "C" H 10450 3000 50  0000 L CNN
+	1    10400 3100
+	1    0    0    -1
+$EndComp
+Text GLabel 2500 4800 0    50   Input ~ 0
+/TRST
 Text GLabel 6800 2700 2    50   Input ~ 0
 RX0
@@
 $EndComp
 $Comp
-L GND #PWR044
+L GND #PWR046
 U 1 1 4BF0021F
 P 9000 5000
-F 0 "#PWR044" H 9000 5000 30  0001 C CNN
+F 0 "#PWR046" H 9000 5000 30  0001 C CNN
 F 1 "GND" H 9000 4930 30  0001 C CNN
 	1    9000 5000
@@
 $EndComp
 $Comp
-L GND #PWR045
+L GND #PWR047
 U 1 1 4BEFBCAA
 P 1000 6850
-F 0 "#PWR045" H 1000 6850 30  0001 C CNN
+F 0 "#PWR047" H 1000 6850 30  0001 C CNN
 F 1 "GND" H 1000 6780 30  0001 C CNN
 	1    1000 6850
@@
 CIC_MCLR
 $Comp
-L GND #PWR046
+L GND #PWR048
 U 1 1 4BEECBF1
 P 2900 6850
-F 0 "#PWR046" H 2900 6850 30  0001 C CNN
+F 0 "#PWR048" H 2900 6850 30  0001 C CNN
 F 1 "GND" H 2900 6780 30  0001 C CNN
 	1    2900 6850
@@
 $EndComp
 $Comp
-L GND #PWR047
+L GND #PWR049
 U 1 1 4BEECBEF
 P 2300 6850
-F 0 "#PWR047" H 2300 6850 30  0001 C CNN
+F 0 "#PWR049" H 2300 6850 30  0001 C CNN
 F 1 "GND" H 2300 6780 30  0001 C CNN
 	1    2300 6850
@@
 $EndComp
 $Comp
-L GND #PWR048
+L GND #PWR050
 U 1 1 4BEECBEE
 P 2000 6850
-F 0 "#PWR048" H 2000 6850 30  0001 C CNN
+F 0 "#PWR050" H 2000 6850 30  0001 C CNN
 F 1 "GND" H 2000 6780 30  0001 C CNN
 	1    2000 6850
@@
 $EndComp
 $Comp
-L GND #PWR049
+L GND #PWR051
 U 1 1 4BEECBE5
 P 1400 6850
-F 0 "#PWR049" H 1400 6850 30  0001 C CNN
+F 0 "#PWR051" H 1400 6850 30  0001 C CNN
 F 1 "GND" H 1400 6780 30  0001 C CNN
 	1    1400 6850
@@
 $EndComp
 $Comp
-L GND #PWR050
+L GND #PWR052
 U 1 1 4BB8BBE8
-P 10200 3900
-F 0 "#PWR050" H 10200 3900 30  0001 C CNN
-F 1 "GND" H 10200 3830 30  0001 C CNN
-	1    10200 3900
-	1    0    0    -1
-$EndComp
-$Comp
-L +3.3V #PWR051
+P 10400 3900
+F 0 "#PWR052" H 10400 3900 30  0001 C CNN
+F 1 "GND" H 10400 3830 30  0001 C CNN
+	1    10400 3900
+	1    0    0    -1
+$EndComp
+$Comp
+L +3.3V #PWR053
 U 1 1 4BB8BBD6
-P 10200 2650
-F 0 "#PWR051" H 10200 2610 30  0001 C CNN
-F 1 "+3.3V" H 10200 2760 30  0000 C CNN
-	1    10200 2650
-	1    0    0    -1
-$EndComp
-$Comp
-L +3.3V #PWR052
+P 10400 2650
+F 0 "#PWR053" H 10400 2610 30  0001 C CNN
+F 1 "+3.3V" H 10400 2760 30  0000 C CNN
+	1    10400 2650
+	1    0    0    -1
+$EndComp
+$Comp
+L +3.3V #PWR054
 U 1 1 4BB8BB64
 P 4450 1450
-F 0 "#PWR052" H 4450 1410 30  0001 C CNN
+F 0 "#PWR054" H 4450 1410 30  0001 C CNN
 F 1 "+3.3V" H 4450 1560 30  0000 C CNN
 	1    4450 1450
@@
 $EndComp
 $Comp
-L GND #PWR053
+L GND #PWR055
 U 1 1 4BB8BB56
 P 4250 6850
-F 0 "#PWR053" H 4250 6850 30  0001 C CNN
+F 0 "#PWR055" H 4250 6850 30  0001 C CNN
 F 1 "GND" H 4250 6780 30  0001 C CNN
 	1    4250 6850
@@
 $EndComp
 $Comp
-L +BATT #PWR054
+L +BATT #PWR056
 U 1 1 4BB8AE61
 P 4150 1450
-F 0 "#PWR054" H 4150 1400 20  0001 C CNN
+F 0 "#PWR056" H 4150 1400 20  0001 C CNN
 F 1 "+BATT" H 4150 1550 30  0000 C CNN
 	1    4150 1450
@@
 $EndComp
 $Comp
-L +3.3V #PWR055
+L +3.3V #PWR057
 U 1 1 4BB8AE12
 P 5050 1450
-F 0 "#PWR055" H 5050 1410 30  0001 C CNN
+F 0 "#PWR057" H 5050 1410 30  0001 C CNN
 F 1 "+3.3V" H 5050 1560 30  0000 C CNN
 	1    5050 1450
@@
 $EndComp
 $Comp
-L GND #PWR056
+L GND #PWR058
 U 1 1 4BAF2DEB
 P 4450 6850
-F 0 "#PWR056" H 4450 6850 30  0001 C CNN
+F 0 "#PWR058" H 4450 6850 30  0001 C CNN
 F 1 "GND" H 4450 6780 30  0001 C CNN
 	1    4450 6850
@@
 $EndComp
 $Comp
-L GND #PWR057
+L GND #PWR059
 U 1 1 4BAF2DE3
 P 4900 6850
-F 0 "#PWR057" H 4900 6850 30  0001 C CNN
+F 0 "#PWR059" H 4900 6850 30  0001 C CNN
 F 1 "GND" H 4900 6780 30  0001 C CNN
 	1    4900 6850

Commit message: pcb wip
Parts:
- added D2: BusyLED, symbol LED
- added D3: RdyLED, symbol LED
- added R5, R6: 100, symbol R
- added R7, R8: 270, symbol R
Connections:
- net +3.3V: now also D2.1 (A), D3.1 (A)
- net CCLK: now also R8.1; no longer U11.40 (P0[11]/RXD2/SCL2/MAT3[1])
- net PROG_B: now also R7.2; no longer U11.65 (RX_MCLK/MAT2[0]/TXD3/P4[28])
- net at U11.59 (PWM1[2]/RXD1/P2[1]): now also R6.1
- net at U11.60 (PWM1[1]/TXD1/P2[0]): now also R5.1
- new net: R8.2, U11.40 (P0[11]/RXD2/SCL2/MAT3[1])
- new net: R7.1, U11.65 (RX_MCLK/MAT2[0]/TXD3/P4[28])
- new net: D2.2 (K), R6.2
- new net: D3.2 (K), R5.2
Other:
- note removed: "LEDs"
Changed lines of the file:
@@
-EESchema Schematic File Version 2  date Fri 21 May 2010 07:28:17 PM CEST
+EESchema Schematic File Version 2  date Sun 23 May 2010 01:25:36 AM CEST
 LIBS:power
 LIBS:device
@@
 Sheet 4 6
 Title "sd2snes Mark II"
-Date "21 may 2010"
+Date "22 may 2010"
 Rev "A"
 Comp "Maximilian Rehkopf"
@@
 Comment4 ""
 $EndDescr
+Wire Wire Line
+	7300 3300 7550 3300
+Connection ~ 1050 2350
+Wire Wire Line
+	1200 2450 1200 2350
+Wire Wire Line
+	1200 2350 900  2350
+Wire Wire Line
+	3000 3100 1900 3100
+Wire Wire Line
+	1400 3100 900  3100
+Wire Wire Line
+	900  3100 900  2850
 Connection ~ 8100 6850
 Wire Wire Line
@@
 Connection ~ 7600 6850
 Wire Wire Line
-	7850 6850 7850 6750
+	7850 6750 7850 6850
 Connection ~ 7850 6250
 Wire Wire Line
 	8100 6250 8100 6350
 Wire Wire Line
-	7600 6350 7600 6150
+	7600 6150 7600 6350
 Wire Wire Line
 	3000 4800 2500 4800
@@
 	9000 4600 9100 4600
 Wire Wire Line
-	9100 4350 7550 4350
-Wire Wire Line
-	7550 4350 7550 4200
-Wire Wire Line
-	7550 4200 6500 4200
+	9100 4350 8200 4350
+Wire Wire Line
+	8200 4350 8200 4200
+Wire Wire Line
+	8200 4200 6500 4200
 Wire Wire Line
 	1000 5400 1000 6850
@@
 	3000 4600 2500 4600
 Wire Wire Line
-	6500 4500 6800 4500
-Wire Wire Line
 	3000 4200 2500 4200
 Wire Wire Line
 	6500 3200 6800 3200
 Wire Wire Line
-	6500 3100 8850 3100
+	8850 3100 6500 3100
 Wire Wire Line
 	8850 3200 7550 3200
@@
 	8750 2650 8750 2900
 Wire Wire Line
-	6500 2900 8850 2900
+	8850 2900 6500 2900
 Connection ~ 10400 3500
 Wire Wire Line
@@
 	7550 2800 6500 2800
 Wire Wire Line
-	8850 3000 6500 3000
+	6500 3000 8850 3000
 Wire Wire Line
 	8650 2650 8650 3000
@@
 	6800 3800 6500 3800
 Wire Wire Line
-	6500 4400 6800 4400
-Wire Wire Line
 	3000 4500 2500 4500
 Wire Wire Line
@@
 	1000 5200 3000 5200
 Wire Wire Line
-	6500 4100 7450 4100
-Wire Wire Line
-	7450 4100 7450 4450
-Wire Wire Line
-	7450 4450 9100 4450
-Wire Wire Line
-	2800 850  7650 850
-Wire Wire Line
-	7650 850  7650 4200
-Wire Wire Line
-	7650 4200 9100 4200
+	6500 4100 8100 4100
+Wire Wire Line
+	8100 4100 8100 4450
+Wire Wire Line
+	8100 4450 9100 4450
+Wire Wire Line
+	2800 850  8300 850
+Wire Wire Line
+	8300 850  8300 4200
+Wire Wire Line
+	8300 4200 9100 4200
 Wire Wire Line
 	9100 4700 9000 4700
@@
 	6500 2700 6800 2700
 Wire Wire Line
-	7600 6750 7600 6950
+	7600 6950 7600 6750
 Wire Wire Line
 	7850 6250 7850 6350
@@
 	8100 6850 8100 6750
 Connection ~ 7850 6850
-$Comp
-L GND #PWR044
+Wire Wire Line
+	1200 2850 1200 3000
+Wire Wire Line
+	1200 3000 1400 3000
+Wire Wire Line
+	1900 3000 3000 3000
+Wire Wire Line
+	1050 2250 1050 2350
+Wire Wire Line
+	900  2350 900  2450
+Wire Wire Line
+	1750 4200 2000 4200
+$Comp
+L R R8
+U 1 1 4BF850D1
+P 7050 3300
+F 0 "R8" V 7000 3550 50  0000 C CNN
+F 1 "270" V 7050 3300 50  0000 C CNN
+	1    7050 3300
+	0    1    1    0
+$EndComp
+$Comp
+L R R7
+U 1 1 4BF850A9
+P 2250 4200
+F 0 "R7" V 2150 4200 50  0000 C CNN
+F 1 "270" V 2250 4200 50  0000 C CNN
+	1    2250 4200
+	0    1    1    0
+$EndComp
+$Comp
+L +3.3V #PWR044
+U 1 1 4BF84ABB
+P 1050 2250
+F 0 "#PWR044" H 1050 2210 30  0001 C CNN
+F 1 "+3.3V" H 1050 2360 30  0000 C CNN
+	1    1050 2250
+	-1   0    0    -1
+$EndComp
+$Comp
+L R R6
+U 1 1 4BF847B1
+P 1650 3100
+F 0 "R6" V 1730 3100 50  0000 C CNN
+F 1 "100" V 1650 3100 50  0000 C CNN
+	1    1650 3100
+	0    1    1    0
+$EndComp
+$Comp
+L R R5
+U 1 1 4BF847A7
+P 1650 3000
+F 0 "R5" V 1550 3000 50  0000 C CNN
+F 1 "100" V 1650 3000 50  0000 C CNN
+	1    1650 3000
+	0    1    1    0
+$EndComp
+$Comp
+L LED D3
+U 1 1 4BF8328D
+P 1200 2650
+F 0 "D3" H 1200 2750 50  0000 C CNN
+F 1 "RdyLED" H 1200 2550 50  0000 C CNN
+	1    1200 2650
+	0    -1   1    0
+$EndComp
+$Comp
+L LED D2
+U 1 1 4BF8324A
+P 900 2650
+F 0 "D2" H 900 2750 50  0000 C CNN
+F 1 "BusyLED" H 900 2550 50  0000 C CNN
+	1    900  2650
+	0    -1   1    0
+$EndComp
+$Comp
+L GND #PWR045
 U 1 1 4BF6C1FC
 P 7600 6950
-F 0 "#PWR044" H 7600 6950 30  0001 C CNN
+F 0 "#PWR045" H 7600 6950 30  0001 C CNN
 F 1 "GND" H 7600 6880 30  0001 C CNN
 	1    7600 6950
@@
 $EndComp
 $Comp
-L +3.3V #PWR045
+L +3.3V #PWR046
 U 1 1 4BF6C1F7
 P 7600 6150
-F 0 "#PWR045" H 7600 6110 30  0001 C CNN
+F 0 "#PWR046" H 7600 6110 30  0001 C CNN
 F 1 "+3.3V" H 7600 6260 30  0000 C CNN
 	1    7600 6150
@@
 $EndComp
 $Comp
-L GND #PWR046
+L GND #PWR047
 U 1 1 4BF0021F
 P 9000 5000
-F 0 "#PWR046" H 9000 5000 30  0001 C CNN
+F 0 "#PWR047" H 9000 5000 30  0001 C CNN
 F 1 "GND" H 9000 4930 30  0001 C CNN
 	1    9000 5000
@@
 $EndComp
 $Comp
-L GND #PWR047
+L GND #PWR048
 U 1 1 4BEFBCAA
 P 1000 6850
-F 0 "#PWR047" H 1000 6850 30  0001 C CNN
+F 0 "#PWR048" H 1000 6850 30  0001 C CNN
 F 1 "GND" H 1000 6780 30  0001 C CNN
 	1    1000 6850
@@
 Text GLabel 2500 4500 0    50   Output ~ 0
 MCU_TDO
-Text Notes 6850 4500 0    50   ~ 0
-LEDs
-Text GLabel 2500 4200 0    50   Output ~ 0
+Text GLabel 1750 4200 0    50   Output ~ 0
 PROG_B
 Text GLabel 6800 3200 2    50   Output ~ 0
 FPGA_CLK
-Text GLabel 6800 3300 2    50   Output ~ 0
+Text GLabel 7550 3300 2    50   Output ~ 0
 CCLK
 Text GLabel 6800 3800 2    50   Input ~ 0
@@
 CIC_MCLR
 $Comp
-L GND #PWR048
+L GND #PWR049
 U 1 1 4BEECBF1
 P 2900 6850
-F 0 "#PWR048" H 2900 6850 30  0001 C CNN
+F 0 "#PWR049" H 2900 6850 30  0001 C CNN
 F 1 "GND" H 2900 6780 30  0001 C CNN
 	1    2900 6850
@@
 $EndComp
 $Comp
-L GND #PWR049
+L GND #PWR050
 U 1 1 4BEECBEF
 P 2300 6850
-F 0 "#PWR049" H 2300 6850 30  0001 C CNN
+F 0 "#PWR050" H 2300 6850 30  0001 C CNN
 F 1 "GND" H 2300 6780 30  0001 C CNN
 	1    2300 6850
@@
 $EndComp
 $Comp
-L GND #PWR050
+L GND #PWR051
 U 1 1 4BEECBEE
 P 2000 6850
-F 0 "#PWR050" H 2000 6850 30  0001 C CNN
+F 0 "#PWR051" H 2000 6850 30  0001 C CNN
 F 1 "GND" H 2000 6780 30  0001 C CNN
 	1    2000 6850
@@
 $EndComp
 $Comp
-L GND #PWR051
+L GND #PWR052
 U 1 1 4BEECBE5
 P 1400 6850
-F 0 "#PWR051" H 1400 6850 30  0001 C CNN
+F 0 "#PWR052" H 1400 6850 30  0001 C CNN
 F 1 "GND" H 1400 6780 30  0001 C CNN
 	1    1400 6850
@@
 $EndComp
 $Comp
-L GND #PWR052
+L GND #PWR053
 U 1 1 4BB8BBE8
 P 10400 3900
-F 0 "#PWR052" H 10400 3900 30  0001 C CNN
+F 0 "#PWR053" H 10400 3900 30  0001 C CNN
 F 1 "GND" H 10400 3830 30  0001 C CNN
 	1    10400 3900
@@
 $EndComp
 $Comp
-L +3.3V #PWR053
+L +3.3V #PWR054
 U 1 1 4BB8BBD6
 P 10400 2650
-F 0 "#PWR053" H 10400 2610 30  0001 C CNN
+F 0 "#PWR054" H 10400 2610 30  0001 C CNN
 F 1 "+3.3V" H 10400 2760 30  0000 C CNN
 	1    10400 2650
@@
 $EndComp
 $Comp
-L +3.3V #PWR054
+L +3.3V #PWR055
 U 1 1 4BB8BB64
 P 4450 1450
-F 0 "#PWR054" H 4450 1410 30  0001 C CNN
+F 0 "#PWR055" H 4450 1410 30  0001 C CNN
 F 1 "+3.3V" H 4450 1560 30  0000 C CNN
 	1    4450 1450
@@
 $EndComp
 $Comp
-L GND #PWR055
+L GND #PWR056
 U 1 1 4BB8BB56
 P 4250 6850
-F 0 "#PWR055" H 4250 6850 30  0001 C CNN
+F 0 "#PWR056" H 4250 6850 30  0001 C CNN
 F 1 "GND" H 4250 6780 30  0001 C CNN
 	1    4250 6850
@@
 $EndComp
 $Comp
-L +BATT #PWR056
+L +BATT #PWR057
 U 1 1 4BB8AE61
 P 4150 1450
-F 0 "#PWR056" H 4150 1400 20  0001 C CNN
+F 0 "#PWR057" H 4150 1400 20  0001 C CNN
 F 1 "+BATT" H 4150 1550 30  0000 C CNN
 	1    4150 1450
@@
 $EndComp
 $Comp
-L +3.3V #PWR057
+L +3.3V #PWR058
 U 1 1 4BB8AE12
 P 5050 1450
-F 0 "#PWR057" H 5050 1410 30  0001 C CNN
+F 0 "#PWR058" H 5050 1410 30  0001 C CNN
 F 1 "+3.3V" H 5050 1560 30  0000 C CNN
 	1    5050 1450
@@
 $EndComp
 $Comp
-L GND #PWR058
+L GND #PWR059
 U 1 1 4BAF2DEB
 P 4450 6850
-F 0 "#PWR058" H 4450 6850 30  0001 C CNN
+F 0 "#PWR059" H 4450 6850 30  0001 C CNN
 F 1 "GND" H 4450 6780 30  0001 C CNN
 	1    4450 6850
@@
 $EndComp
 $Comp
-L GND #PWR059
+L GND #PWR060
 U 1 1 4BAF2DE3
 P 4900 6850
-F 0 "#PWR059" H 4900 6850 30  0001 C CNN
+F 0 "#PWR060" H 4900 6850 30  0001 C CNN
 F 1 "GND" H 4900 6780 30  0001 C CNN
 	1    4900 6850

Commit message: pcb wip
Parts:
- removed P1: CONN_14, symbol CONN_14
- added P1: CONN_8X2, symbol CONN_8X2
Connections:
- net at U11.55 (PWM1[4]/DCD1/TRACEDATA[2]/P2[3]): now also J2.WP (WPROT)
- net at U11.58 (PWM1[3]/CTS1/TRACEDATA[3]/P2[2]): now also J2.DT (DETECT)
Other:
- moved on the sheet: C40, C41, C42, C43
Changed lines of the file:
@@
-EESchema Schematic File Version 2  date Sun 23 May 2010 01:25:36 AM CEST
+EESchema Schematic File Version 2  date Sun 23 May 2010 11:04:23 PM CEST
 LIBS:power
 LIBS:device
@@
 Sheet 4 6
 Title "sd2snes Mark II"
-Date "22 may 2010"
+Date "23 may 2010"
 Rev "A"
 Comp "Maximilian Rehkopf"
@@
 Comment4 ""
 $EndDescr
+$Comp
+L CONN_8X2 P1
+U 1 1 4BF950B0
+P 9650 6100
+F 0 "P1" H 9650 6550 60  0000 C CNN
+F 1 "CONN_8X2" V 9650 6100 50  0000 C CNN
+	1    9650 6100
+	1    0    0    -1
+$EndComp
+Wire Wire Line
+	8850 3400 8250 3400
+Wire Wire Line
+	3000 3300 2600 3300
+Wire Wire Line
+	2600 3300 2600 850
+Wire Wire Line
+	2600 850  8250 850
+Wire Wire Line
+	8250 850  8250 3400
 Wire Wire Line
 	7300 3300 7550 3300
@@
 Wire Wire Line
 	900  3100 900  2850
-Connection ~ 8100 6850
-Wire Wire Line
-	8350 6750 8350 6850
-Wire Wire Line
-	8350 6850 7600 6850
-Connection ~ 7600 6850
-Wire Wire Line
-	7850 6750 7850 6850
-Connection ~ 7850 6250
-Wire Wire Line
-	8100 6250 8100 6350
-Wire Wire Line
-	7600 6150 7600 6350
+Connection ~ 6150 7600
+Wire Wire Line
+	6400 7500 6400 7600
+Wire Wire Line
+	6400 7600 5650 7600
+Connection ~ 5650 7600
+Wire Wire Line
+	5900 7500 5900 7600
+Connection ~ 5900 7000
+Wire Wire Line
+	6150 7000 6150 7100
+Wire Wire Line
+	5650 6900 5650 7100
 Wire Wire Line
 	3000 4800 2500 4800
@@
 	9000 4600 9100 4600
 Wire Wire Line
-	9100 4350 8200 4350
-Wire Wire Line
-	8200 4350 8200 4200
-Wire Wire Line
-	8200 4200 6500 4200
+	9100 4350 7950 4350
+Wire Wire Line
+	7950 4350 7950 4200
+Wire Wire Line
+	7950 4200 6500 4200
 Wire Wire Line
 	1000 5400 1000 6850
@@
 	3000 2700 2800 2700
 Wire Wire Line
-	2800 2700 2800 850
+	2800 2700 2800 1050
 Wire Wire Line
 	3000 4000 2500 4000
@@
 	1000 5200 3000 5200
 Wire Wire Line
-	6500 4100 8100 4100
-Wire Wire Line
-	8100 4100 8100 4450
-Wire Wire Line
-	8100 4450 9100 4450
-Wire Wire Line
-	2800 850  8300 850
-Wire Wire Line
-	8300 850  8300 4200
-Wire Wire Line
-	8300 4200 9100 4200
+	6500 4100 7850 4100
+Wire Wire Line
+	7850 4100 7850 4450
+Wire Wire Line
+	7850 4450 9100 4450
+Wire Wire Line
+	2800 1050 8050 1050
+Wire Wire Line
+	8050 1050 8050 4200
+Wire Wire Line
+	8050 4200 9100 4200
 Wire Wire Line
 	9100 4700 9000 4700
@@
 	6500 2700 6800 2700
 Wire Wire Line
-	7600 6950 7600 6750
-Wire Wire Line
-	7850 6250 7850 6350
-Connection ~ 7600 6250
-Wire Wire Line
-	7600 6250 8350 6250
-Wire Wire Line
-	8350 6250 8350 6350
-Connection ~ 8100 6250
-Wire Wire Line
-	8100 6850 8100 6750
-Connection ~ 7850 6850
+	5650 7700 5650 7500
+Wire Wire Line
+	5900 7000 5900 7100
+Connection ~ 5650 7000
+Wire Wire Line
+	5650 7000 6400 7000
+Wire Wire Line
+	6400 7000 6400 7100
+Connection ~ 6150 7000
+Wire Wire Line
+	6150 7600 6150 7500
+Connection ~ 5900 7600
 Wire Wire Line
 	1200 2850 1200 3000
@@
 Wire Wire Line
 	1750 4200 2000 4200
+Wire Wire Line
+	3000 3200 2700 3200
+Wire Wire Line
+	2700 3200 2700 950
+Wire Wire Line
+	2700 950  8150 950
+Wire Wire Line
+	8150 950  8150 3500
+Wire Wire Line
+	8150 3500 8850 3500
 $Comp
 L R R8
@@
 L GND #PWR045
 U 1 1 4BF6C1FC
-P 7600 6950
-F 0 "#PWR045" H 7600 6950 30  0001 C CNN
-F 1 "GND" H 7600 6880 30  0001 C CNN
-	1    7600 6950
+P 5650 7700
+F 0 "#PWR045" H 5650 7700 30  0001 C CNN
+F 1 "GND" H 5650 7630 30  0001 C CNN
+	1    5650 7700
 	1    0    0    -1
 $EndComp
@@
 L +3.3V #PWR046
 U 1 1 4BF6C1F7
-P 7600 6150
-F 0 "#PWR046" H 7600 6110 30  0001 C CNN
-F 1 "+3.3V" H 7600 6260 30  0000 C CNN
-	1    7600 6150
+P 5650 6900
+F 0 "#PWR046" H 5650 6860 30  0001 C CNN
+F 1 "+3.3V" H 5650 7010 30  0000 C CNN
+	1    5650 6900
 	-1   0    0    -1
 $EndComp
@@
 L C C43
 U 1 1 4BF6BFE6
-P 8350 6550
-F 0 "C43" H 8400 6650 50  0000 L CNN
-F 1 "C" H 8400 6450 50  0000 L CNN
-	1    8350 6550
+P 6400 7300
+F 0 "C43" H 6450 7400 50  0000 L CNN
+F 1 "C" H 6450 7200 50  0000 L CNN
+	1    6400 7300
 	1    0    0    -1
 $EndComp
@@
 L C C42
 U 1 1 4BF6BFE5
-P 8100 6550
-F 0 "C42" H 8150 6650 50  0000 L CNN
-F 1 "C" H 8150 6450 50  0000 L CNN
-	1    8100 6550
+P 6150 7300
+F 0 "C42" H 6200 7400 50  0000 L CNN
+F 1 "C" H 6200 7200 50  0000 L CNN
+	1    6150 7300
 	1    0    0    -1
 $EndComp
@@
 L C C41
 U 1 1 4BF6BFE2
-P 7850 6550
-F 0 "C41" H 7900 6650 50  0000 L CNN
-F 1 "C" H 7900 6450 50  0000 L CNN
-	1    7850 6550
+P 5900 7300
+F 0 "C41" H 5950 7400 50  0000 L CNN
+F 1 "C" H 5950 7200 50  0000 L CNN
+	1    5900 7300
 	1    0    0    -1
 $EndComp
@@
 L C C40
 U 1 1 4BF6BFE1
-P 7600 6550
-F 0 "C40" H 7650 6650 50  0000 L CNN
-F 1 "C" H 7650 6450 50  0000 L CNN
-	1    7600 6550
+P 5650 7300
+F 0 "C40" H 5700 7400 50  0000 L CNN
+F 1 "C" H 5700 7200 50  0000 L CNN
+	1    5650 7300
 	1    0    0    -1
 $EndComp
@@
 CIC_DATA1
 $Comp
-L CONN_14 P1
-U 1 1 4BF3C8DA
-P 10400 6050
-F 0 "P1" V 10370 6050 60  0000 C CNN
-F 1 "CONN_14" V 10480 6050 60  0000 C CNN
-	1    10400 6050
-	1    0    0    -1
-$EndComp
-$Comp
 L GND #PWR047

Commit message: pcb wip
Connections:
- net +3.3V: now also P1.1
- net /TRST: now also P1.9
- net EXT_TDI: now also P1.11
- net GND: now also P1.3
- net INIT_B+MCU_/IRQ: now also P1.4
- net RX0: now also P1.13
- net TCK: now also P1.8
- net TMS: now also P1.10
- net TX0: now also P1.14
- net /RESET: now reaches P2.2 (PM), U11.14 (/RESET)
- net /RESET: now also P1.5
- net RX3: now reaches U11.6 (P0[26]/AD0[3]/AOUT/RXD3)
- net RX3: now also P1.7
- net TX3: now reaches U11.7 (P0[25]/AD0[2]/TXD3)
- net TX3: now also P1.6
- net EXT_TDO: now reaches P1.12
- net +5V: now reaches P1.2
- no-connect marks 0 -> 2
Other:
- moved on the sheet: C40, C41, C42, C43
