File: pcb/kicad/mcu.sch (KiCad schematic (older format))
At the start: 23 parts, among them J2 SD_CARD, J3 USB_MINIB, P1 CONN_8X2, P2 CONN_2, U11 LPC1754, X1 12MHz, X2 32.768kHz

Commit message: pcb wip?
Parts:
- added C62: 100n, symbol C
- added R14: 10k, symbol R
- C40, C41, C42, C43, C44: value C -> 100n
Connections:
- wire segments 146 -> 150

Commit message: pcb+schem wip
Parts:
- R5, R6: value 100 -> 680
Other:
- note added: "2mA low current LEDs"
- note added: "MCU, SD, debug"
- note added: "Reset button"
Changed lines of the file:
@@
-EESchema Schematic File Version 2  date Wed 02 Jun 2010 02:08:21 PM CEST
+EESchema Schematic File Version 2  date Fri 04 Jun 2010 01:55:30 AM CEST
 LIBS:power
 LIBS:device
@@
 Sheet 4 6
 Title "sd2snes Mark II"
-Date "2 jun 2010"
+Date "3 jun 2010"
 Rev "A"
 Comp "Maximilian Rehkopf"
@@
 Comment4 ""
 $EndDescr
+Text Notes 550  7700 0    250  ~ 50
+MCU, SD, debug
+Text Notes 500  5050 0    50   ~ 0
+Reset button
 Connection ~ 1000 5950
 Wire Wire Line
@@
 Wire Wire Line
 	1200 5400 1200 5100
+Text Notes 650  3250 0    50   ~ 0
+2mA low current LEDs
 $Comp
 L C C62
@@
 P 1650 3100
 F 0 "R6" V 1730 3100 50  0000 C CNN
-F 1 "100" V 1650 3100 50  0000 C CNN
+F 1 "680" V 1650 3100 50  0000 C CNN
 	1    1650 3100
 	0    1    1    0
@@
 P 1650 3000
 F 0 "R5" V 1550 3000 50  0000 C CNN
-F 1 "100" V 1650 3000 50  0000 C CNN
+F 1 "680" V 1650 3000 50  0000 C CNN
 	1    1650 3000
 	0    1    1    0

Commit message: pcb wip
Parts:
- removed P1: CONN_8X2, symbol CONN_8X2
- added P1: CONN_7X2, symbol CONN_7X2
- D2: value BusyLED -> LED 2mA 1.7V, red
- D3: value RdyLED -> LED 2mA 1.9V, green
Connections:
- wire segments 150 -> 187
- no-connect marks 2 -> 0
Other:
- moved on the sheet: C34, C35, C36, C37, C40, C41, C42, C43, C44, C62, D2, D3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

Commit message: pcb wip
Parts:
- added D4: LED 2mA 1.7V, red, symbol LED
- added R15: 680, symbol R
- D2: value LED 2mA 1.7V, red -> LED 2mA 1.8V, yellow
Connections:
- net +3.3V: now also D4.1 (A)
- net at U11.54 (PWM1[5]/DSR1/TRACEDATA[1]/P2[4]): now also J2.WP (WPROT)
- net at U11.55 (PWM1[4]/DCD1/TRACEDATA[2]/P2[3]): now also J2.DT (DETECT); no longer J2.WP (WPROT)
- net at U11.58 (PWM1[3]/CTS1/TRACEDATA[3]/P2[2]): now also R15.1; no longer J2.DT (DETECT)
- new net: D4.2 (K), R15.2
Other:
- moved on the sheet: D2, D3, R5, R6

Commit message: pcb wip
Parts:
- C44: value 100n -> 10u
Changed lines of the file:
@@
-EESchema Schematic File Version 2  date Tue 08 Jun 2010 04:15:56 AM CEST
+EESchema Schematic File Version 2  date Thu 10 Jun 2010 11:56:43 PM CEST
 LIBS:power
 LIBS:device
@@
 Sheet 4 6
 Title "sd2snes Mark II"
-Date "8 jun 2010"
+Date "10 jun 2010"
 Rev "A"
 Comp "Maximilian Rehkopf"
@@
 P 10600 3100
 F 0 "C44" H 10650 3200 50  0000 L CNN
-F 1 "100n" H 10650 3000 50  0000 L CNN
+F 1 "10u" H 10650 3000 50  0000 L CNN
 	1    10600 3100
 	1    0    0    -1

Commit message: pcb wip
Parts:
- added C63: 100n, SM0805_FIXEDMASK, symbol C
- C34, C35, C36, C37, C40, C41, C42, C43, C44, C62, R13, R14, R15, R5, R6, R7, R8: footprint (none) -> SM0805_FIXEDMASK
- D2, D3, D4: footprint (none) -> LED-3MM-FIXED
- J2: footprint (none) -> SD-RSMT-2-MQ-WF
- J3: footprint (none) -> USB-MINIB-THT
- P1: footprint (none) -> pin_array_7x2
- P2: footprint (none) -> PIN_ARRAY_2X1
- U11: footprint (none) -> LQFP80-.5
- X1: footprint (none) -> XTAL_SMD_05032
- X2: footprint (none) -> XTAL_SMD_05019
Connections:
- net +3.3V: now also C63.1
- net GND: now also C63.2
- net DIN+MCU_/OVR: now reaches U11.50 (TXD2/P2[8])
