File: pcb/kicad/pwr_misc.sch (KiCad schematic (older format))
At the start: 17 parts, among them U10 MCP1824-2.5, U14 CS4344, U15 PIC12F629, U7 LT1117-3.3, U8 LT1117-1.2, U9 MCP1824-1.8

Commit message: pcb wip
Parts:
- added C45, C47, C49: 3.3u, symbol C
- added C46, C51: 100n, symbol C
- added C48, C50: 10u, symbol C
- added R10, R12: 470, symbol R
- added R11, R9: 10k, symbol R
Connections:
- net GND: now also C46.2, C48.2, C49.2, C50.2, C51.2, R11.2, R9.2
- net at U14.10 (AOUTR): now also C45.2
- net at U14.5 (VQ): now also C50.1, C51.1
- net at U14.6 (FILT): now also C48.1
- net at U14.7 (AOUTL): now also C47.2
- new net: C47.1, R11.1, R12.2
- new net: C45.1, R10.2, R9.1
- new net AUDIO_L: C49.1, R12.1
- new net AUDIO_R: C46.1, R10.1
Other:
- moved on the sheet: BT1, C33, U14
