File: pcb/kicad/pwr_misc.sch (KiCad schematic (older format))
At the start: 28 parts, among them U10 MCP1824-2.5, U14 CS4344, U15 PIC12F629, U7 LT1117-3.3, U8 LT1117-1.2, U9 MCP1824-1.8

Commit message: pcb wip (use switching regulator?)
Parts:
- removed C1, C2: 10u, symbol C
- removed C5, C6: 100u, symbol CP1
- removed U7: LT1117-3.3, symbol LT1117
- removed U8: LT1117-1.2, symbol LT1117
- added C58, C59, C61: 4.7u, symbol C
- added C60: 10n, symbol C
- added L1, L2: 1uH, symbol INDUCTOR
- added U16: MIC23250_FIXOUT, symbol MIC23250_FIXOUT
Connections:
- wire segments 88 -> 92

Commit message: pcb wip?
Connections:
- net REG_SW1: now reaches L1.2, U16.4 (SW1)
- net REG_SW2: now reaches L2.1, U16.7 (SW2)
Changed lines of the file:
@@
-EESchema Schematic File Version 2  date Wed 02 Jun 2010 03:59:20 AM CEST
+EESchema Schematic File Version 2  date Wed 02 Jun 2010 02:08:21 PM CEST
 LIBS:power
 LIBS:device
@@
 Comment4 ""
 $EndDescr
-$Comp
-L +3.3V #PWR?
+Text Label 2800 2400 0    50   ~ 0
+REG_SW1
+Text Label 4450 2400 0    50   ~ 0
+REG_SW2
+$Comp
+L +3.3V #PWR066
 U 1 1 4C05BAF5
 P 5450 2400
-F 0 "#PWR?" H 5450 2360 30  0001 C CNN
+F 0 "#PWR066" H 5450 2360 30  0001 C CNN
 F 1 "+3.3V" H 5450 2510 30  0000 C CNN
 	1    5450 2400
@@
 $EndComp
 $Comp
-L +1.2V #PWR?
+L +1.2V #PWR067
 U 1 1 4C05BAEC
 P 1850 2400
-F 0 "#PWR?" H 1850 2540 20  0001 C CNN
+F 0 "#PWR067" H 1850 2540 20  0001 C CNN
 F 1 "+1.2V" H 1850 2510 30  0000 C CNN
 	1    1850 2400
@@
 	7800 5400 7700 5400
 Wire Wire Line
-	10000 5200 10000 5000
+	10000 5000 10000 5200
 Connection ~ 10000 5700
 Wire Wire Line
@@
 	1750 6450 1850 6450
 Wire Wire Line
-	3950 4450 3950 4650
-Wire Wire Line
-	3950 4650 3250 4650
+	3950 4650 3950 4450
+Wire Wire Line
+	3250 4650 3950 4650
 Wire Wire Line
 	1850 4650 1150 4650
@@
 Connection ~ 1750 4650
 Wire Wire Line
-	1150 6050 1150 6250
-Wire Wire Line
-	1150 6250 1850 6250
+	1150 6250 1150 6050
+Wire Wire Line
+	1850 6250 1150 6250
 Wire Wire Line
 	3250 6250 3950 6250
@@
 	9300 5600 9300 5800
 Wire Wire Line
-	10000 5000 7700 5000
+	7700 5000 10000 5000
 Wire Wire Line
 	9700 5600 9700 5700
@@
 	2750 2400 2900 2400
 Wire Wire Line
-	2000 2400 2000 2600
+	2000 2600 2000 2400
 Wire Wire Line
 	2000 2600 2900 2600
@@
 Connection ~ 2000 2400
 $Comp
-L GND #PWR065
+L GND #PWR068
 U 1 1 4C05AF72
 P 2500 2100
-F 0 "#PWR065" H 2500 2100 30  0001 C CNN
+F 0 "#PWR068" H 2500 2100 30  0001 C CNN
 F 1 "GND" H 2500 2030 30  0001 C CNN
 	1    2500 2100
@@
 $EndComp
 $Comp
-L GND #PWR066
+L GND #PWR069
 U 1 1 4C05ADCE
 P 5300 3500
-F 0 "#PWR066" H 5300 3500 30  0001 C CNN
+F 0 "#PWR069" H 5300 3500 30  0001 C CNN
 F 1 "GND" H 5300 3430 30  0001 C CNN
 	1    5300 3500
@@
 $EndComp
 $Comp
-L GND #PWR067
+L GND #PWR070
 U 1 1 4C05ADC9
 P 2000 3500
-F 0 "#PWR067" H 2000 3500 30  0001 C CNN
+F 0 "#PWR070" H 2000 3500 30  0001 C CNN
 F 1 "GND" H 2000 3430 30  0001 C CNN
 	1    2000 3500
@@
 $EndComp
 $Comp
-L +5V #PWR068
+L +5V #PWR071
 U 1 1 4C05AD31
 P 2000 1300
-F 0 "#PWR068" H 2000 1390 20  0001 C CNN
+F 0 "#PWR071" H 2000 1390 20  0001 C CNN
 F 1 "+5V" H 2000 1390 30  0000 C CNN
 	1    2000 1300
@@
 $EndComp
 $Comp
-L GND #PWR069
+L GND #PWR072
 U 1 1 4C05AD0F
 P 4700 2100
-F 0 "#PWR069" H 4700 2100 30  0001 C CNN
+F 0 "#PWR072" H 4700 2100 30  0001 C CNN
 F 1 "GND" H 4700 2030 30  0001 C CNN
 	1    4700 2100
@@
 $EndComp
 $Comp
-L GND #PWR070
+L GND #PWR073
 U 1 1 4C05A4CA
 P 3750 3500
-F 0 "#PWR070" H 3750 3500 30  0001 C CNN
+F 0 "#PWR073" H 3750 3500 30  0001 C CNN
 F 1 "GND" H 3750 3430 30  0001 C CNN
 	1    3750 3500
@@
 $EndComp
 $Comp
-L GND #PWR071
+L GND #PWR074
 U 1 1 4C05A4C3
 P 3550 3500
-F 0 "#PWR071" H 3550 3500 30  0001 C CNN
+F 0 "#PWR074" H 3550 3500 30  0001 C CNN
 F 1 "GND" H 3550 3430 30  0001 C CNN
 	1    3550 3500
@@
 AUDIO_L
 $Comp
-L GND #PWR072
+L GND #PWR075
 U 1 1 4BF98FD5
 P 9550 6800
-F 0 "#PWR072" H 9550 6800 30  0001 C CNN
+F 0 "#PWR075" H 9550 6800 30  0001 C CNN
 F 1 "GND" H 9550 6730 30  0001 C CNN
 	1    9550 6800
@@
 $EndComp
 $Comp
-L GND #PWR073
+L GND #PWR076
 U 1 1 4BF98FC7
 P 8950 6800
-F 0 "#PWR073" H 8950 6800 30  0001 C CNN
+F 0 "#PWR076" H 8950 6800 30  0001 C CNN
 F 1 "GND" H 8950 6730 30  0001 C CNN
 	1    8950 6800
@@
 AUDIO_R
 $Comp
-L GND #PWR074
+L GND #PWR077
 U 1 1 4BF98F5A
 P 8400 6800
-F 0 "#PWR074" H 8400 6800 30  0001 C CNN
+F 0 "#PWR077" H 8400 6800 30  0001 C CNN
 F 1 "GND" H 8400 6730 30  0001 C CNN
 	1    8400 6800
@@
 $EndComp
 $Comp
-L GND #PWR075
+L GND #PWR078
 U 1 1 4BF98F1F
 P 7800 6800
-F 0 "#PWR075" H 7800 6800 30  0001 C CNN
+F 0 "#PWR078" H 7800 6800 30  0001 C CNN
 F 1 "GND" H 7800 6730 30  0001 C CNN
 	1    7800 6800
@@
 $EndComp
 $Comp
-L GND #PWR076
+L GND #PWR079
 U 1 1 4BF98D19
 P 9300 5800
-F 0 "#PWR076" H 9300 5800 30  0001 C CNN
+F 0 "#PWR079" H 9300 5800 30  0001 C CNN
 F 1 "GND" H 9300 5730 30  0001 C CNN
 	1    9300 5800
@@
 $EndComp
 $Comp
-L GND #PWR077
+L GND #PWR080
 U 1 1 4BF98C9E
 P 10000 5800
-F 0 "#PWR077" H 10000 5800 30  0001 C CNN
+F 0 "#PWR080" H 10000 5800 30  0001 C CNN
 F 1 "GND" H 10000 5730 30  0001 C CNN
 	1    10000 5800
@@
 CIC_CLK
 $Comp
-L +BATT #PWR078
+L +BATT #PWR081
 U 1 1 4BAF2EDB
 P 5050 6400
-F 0 "#PWR078" H 5050 6350 20  0001 C CNN
+F 0 "#PWR081" H 5050 6350 20  0001 C CNN
 F 1 "+BATT" H 5050 6500 30  0000 C CNN
 	1    5050 6400
@@
 $EndComp
 $Comp
-L GND #PWR079
+L GND #PWR082
 U 1 1 4BAF2ED2
 P 6050 6600
-F 0 "#PWR079" H 6050 6600 30  0001 C CNN
+F 0 "#PWR082" H 6050 6600 30  0001 C CNN
 F 1 "GND" H 6050 6530 30  0001 C CNN
 	1    6050 6600
@@
 $EndComp
 $Comp
-L GND #PWR080
+L GND #PWR083
 U 1 1 4BADC749
 P 10300 6950
-F 0 "#PWR080" H 10300 6950 30  0001 C CNN
+F 0 "#PWR083" H 10300 6950 30  0001 C CNN
 F 1 "GND" H 10300 6880 30  0001 C CNN
 	1    10300 6950
@@
 $EndComp
 $Comp
-L +3.3V #PWR081
+L +3.3V #PWR084
 U 1 1 4BADC711
 P 10300 6350
-F 0 "#PWR081" H 10300 6310 30  0001 C CNN
+F 0 "#PWR084" H 10300 6310 30  0001 C CNN
 F 1 "+3.3V" H 10300 6460 30  0000 C CNN
 	1    10300 6350
@@
 $EndComp
 $Comp
-L GND #PWR082
+L GND #PWR085
 U 1 1 4BAD0CFA
 P 7000 6100
-F 0 "#PWR082" H 7000 6100 30  0001 C CNN
+F 0 "#PWR085" H 7000 6100 30  0001 C CNN
 F 1 "GND" H 7000 6030 30  0001 C CNN
 	1    7000 6100
@@
 $EndComp
 $Comp
-L +3.3V #PWR083
+L +3.3V #PWR086
 U 1 1 4BAD0CEA
 P 7000 4350
-F 0 "#PWR083" H 7000 4310 30  0001 C CNN
+F 0 "#PWR086" H 7000 4310 30  0001 C CNN
 F 1 "+3.3V" H 7000 4460 30  0000 C CNN
 	1    7000 4350
@@
 $EndComp
 $Comp
-L GND #PWR084
+L GND #PWR087
 U 1 1 4BADC745
 P 10700 3500
-F 0 "#PWR084" H 10700 3500 30  0001 C CNN
+F 0 "#PWR087" H 10700 3500 30  0001 C CNN
 F 1 "GND" H 10700 3430 30  0001 C CNN
 	1    10700 3500
@@
 $EndComp
 $Comp
-L +5V #PWR085
+L +5V #PWR088
 U 1 1 4BADC709
 P 10700 2900
-F 0 "#PWR085" H 10700 2990 20  0001 C CNN
+F 0 "#PWR088" H 10700 2990 20  0001 C CNN
 F 1 "+5V" H 10700 2990 30  0000 C CNN
 	1    10700 2900
@@
 CIC_CLK
 $Comp
-L GND #PWR086
+L GND #PWR089
 U 1 1 4BAD0C41
 P 9450 2450
-F 0 "#PWR086" H 9450 2450 30  0001 C CNN
+F 0 "#PWR089" H 9450 2450 30  0001 C CNN
 F 1 "GND" H 9450 2380 30  0001 C CNN
 	1    9450 2450
@@
 $EndComp
 $Comp
-L GND #PWR087
+L GND #PWR090
 U 1 1 4BABCB69
 P 3500 5350
-F 0 "#PWR087" H 3500 5350 30  0001 C CNN
+F 0 "#PWR090" H 3500 5350 30  0001 C CNN
 F 1 "GND" H 3500 5280 30  0001 C CNN
 	1    3500 5350
@@
 $EndComp
 $Comp
-L GND #PWR088
+L GND #PWR091
 U 1 1 4BABCB5B
 P 1600 5350
-F 0 "#PWR088" H 1600 5350 30  0001 C CNN
+F 0 "#PWR091" H 1600 5350 30  0001 C CNN
 F 1 "GND" H 1600 5280 30  0001 C CNN
 	1    1600 5350
@@
 $EndComp
 $Comp
-L GND #PWR089
+L GND #PWR092
 U 1 1 4BABCAF4
 P 1600 6950
-F 0 "#PWR089" H 1600 6950 30  0001 C CNN
+F 0 "#PWR092" H 1600 6950 30  0001 C CNN
 F 1 "GND" H 1600 6880 30  0001 C CNN
 	1    1600 6950
@@
 $EndComp
 $Comp
-L GND #PWR090
+L GND #PWR093
 U 1 1 4BABCA9D
 P 3500 6950
-F 0 "#PWR090" H 3500 6950 30  0001 C CNN
+F 0 "#PWR093" H 3500 6950 30  0001 C CNN
 F 1 "GND" H 3500 6880 30  0001 C CNN
 	1    3500 6950
@@
 CIC Clone
 $Comp
-L +5V #PWR091
+L +5V #PWR094
 U 1 1 4BABC073
 P 7300 2250
-F 0 "#PWR091" H 7300 2340 20  0001 C CNN
+F 0 "#PWR094" H 7300 2340 20  0001 C CNN
 F 1 "+5V" H 7300 2340 30  0000 C CNN
 	1    7300 2250
@@
 $EndComp
 $Comp
-L GND #PWR092
+L GND #PWR095
 U 1 1 4B6ED41C
 P 2550 6950
-F 0 "#PWR092" H 2550 6950 30  0001 C CNN
+F 0 "#PWR095" H 2550 6950 30  0001 C CNN
 F 1 "GND" H 2550 6880 30  0001 C CNN
 	1    2550 6950
@@
 $EndComp
 $Comp
-L GND #PWR093
+L GND #PWR096
 U 1 1 4B6ED418
 P 2550 5350
-F 0 "#PWR093" H 2550 5350 30  0001 C CNN
+F 0 "#PWR096" H 2550 5350 30  0001 C CNN
 F 1 "GND" H 2550 5280 30  0001 C CNN
 	1    2550 5350
@@
 $EndComp
 $Comp
-L +3.3V #PWR094
+L +3.3V #PWR097
 U 1 1 4B6ED26C
 P 1150 6050
-F 0 "#PWR094" H 1150 6010 30  0001 C CNN
+F 0 "#PWR097" H 1150 6010 30  0001 C CNN
 F 1 "+3.3V" H 1150 6160 30  0000 C CNN
 	1    1150 6050
@@
 $EndComp
 $Comp
-L +3.3V #PWR095
+L +3.3V #PWR098
 U 1 1 4B6ED268
 P 1150 4450
-F 0 "#PWR095" H 1150 4410 30  0001 C CNN
+F 0 "#PWR098" H 1150 4410 30  0001 C CNN
 F 1 "+3.3V" H 1150 4560 30  0000 C CNN
 	1    1150 4450
@@
 $EndComp
 $Comp
-L +2.5V #PWR096
+L +2.5V #PWR099
 U 1 1 4B6ED246
 P 3950 6050
-F 0 "#PWR096" H 3950 6000 20  0001 C CNN
+F 0 "#PWR099" H 3950 6000 20  0001 C CNN
 F 1 "+2.5V" H 3950 6150 30  0000 C CNN
 	1    3950 6050
@@
 $EndComp
 $Comp
-L +1.8V #PWR097
+L +1.8V #PWR0100
 U 1 1 4B6ED23A
 P 3950 4450
-F 0 "#PWR097" H 3950 4590 20  0001 C CNN
+F 0 "#PWR0100" H 3950 4590 20  0001 C CNN
 F 1 "+1.8V" H 3950 4560 30  0000 C CNN
 	1    3950 4450

Commit message: pcb+schem wip
Other:
- note added: "1.8V LDO"
- note added: "2.5V LDO"
- note added: "3.3V + 1.2V Step-Down"
- note added: "Battery (SRAM + RTC)"
- note added: "Power, DAC, CIC, Batt"
- moved on the sheet: BT1, C32, C33, C45, C46, C47, C48, C49, C50, C51, C58, C59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

Commit message: pcb wip
Parts:
- BT1: footprint (none) -> BT_KEYSTONE_1059_20MM
- C3, C32, C33, C4, C45, C46, C47, C48, C49, C50, C51, C58, C59, C60, C61, C7, C8, R10, R11, R12, R9: footprint (none) -> SM0805_FIXEDMASK
- L1, L2: footprint (none) -> SM1210L
- U10, U9: footprint (none) -> SOT23-5
- U14: footprint (none) -> TSSOP10
- U15: footprint (none) -> SO8N
- U16: footprint (none) -> QFN10-2x2

Commit message: pcb wip
Parts:
- BT1: value BATTERY -> Keystone 1059 / KZH20PCB
- U16: value MIC23250_FIXOUT -> MIC23250-S4YMT
Changed lines of the file:
@@
-EESchema Schematic File Version 2  date Fri 11 Jun 2010 11:43:50 PM CEST
+EESchema Schematic File Version 2  date Sat 12 Jun 2010 06:26:09 PM CEST
 LIBS:power
 LIBS:device
@@
 Sheet 5 6
 Title "sd2snes Mark II"
-Date "11 jun 2010"
+Date "12 jun 2010"
 Rev "A"
 Comp "Maximilian Rehkopf"
@@
 P 2550 2500
 F 0 "U16" H 2550 2600 60  0000 C CNN
-F 1 "MIC23250_FIXOUT" H 2550 2400 60  0000 C CNN
+F 1 "MIC23250-S4YMT" H 2550 2400 60  0000 C CNN
 F 2 "QFN10-2x2" H 2550 2500 60  0001 C CNN
 	1    2550 2500
@@
 P 5800 7000
 F 0 "BT1" H 5800 7200 50  0000 C CNN
-F 1 "BATTERY" H 5800 6810 50  0000 C CNN
+F 1 "Keystone 1059 / KZH20PCB" H 5800 6810 50  0000 C CNN
 F 2 "BT_KEYSTONE_1059_20MM" H 5800 7000 60  0001 C CNN
 	1    5800 7000
