File: pcb/kicad/memory.sch (KiCad schematic (older format))
At the start: 10 parts, among them Q1 NPN, U12 MT45W8MW16, U13 CY62148EV30-BVXI

Commit message: pcb+schem wip
Other:
- note added: "128Mbits 70ns PSRAM (ROM area)"
- note added: "4Mbits 55ns SRAM (battery RAM + custom chip work RAM)"
- note added: "Battery power OE switch"
- note added: "Memory"
- note added: "SRAM battery power"
- note removed: ""ROM""
- note removed: "SRAM"
Changed lines of the file:
@@
-EESchema Schematic File Version 2  date Wed 02 Jun 2010 02:08:21 PM CEST
+EESchema Schematic File Version 2  date Fri 04 Jun 2010 01:55:30 AM CEST
 LIBS:power
 LIBS:device
@@
 Sheet 3 6
 Title "sd2snes Mark II"
-Date "2 jun 2010"
+Date "3 jun 2010"
 Rev "A"
 Comp "Maximilian Rehkopf"
@@
 Comment4 ""
 $EndDescr
+Text Notes 7050 7000 0    250  ~ 50
+Memory
+Text Notes 7300 1300 0    50   ~ 0
+SRAM battery power
+Text Notes 9800 5300 0    50   ~ 0
+Battery power OE switch
 $Comp
 L +3.3V #PWR030
@@
 	1    0    0    -1
 $EndComp
-Text Notes 7100 2400 0    60   ~ 0
-SRAM
-Text Notes 2900 2000 0    60   ~ 0
-"ROM"
+Text Notes 6300 5700 0    60   ~ 0
+4Mbits 55ns SRAM (battery RAM + custom chip work RAM)
+Text Notes 2650 5700 0    60   ~ 0
+128Mbits 70ns PSRAM (ROM area)
 $Comp
 L CY62148EV30-BVXI U13

Commit message: pcb wip
Parts:
- Q1: value NPN -> 2N2222A
Changed lines of the file:
@@
-EESchema Schematic File Version 2  date Tue 08 Jun 2010 04:15:56 AM CEST
+EESchema Schematic File Version 2  date Thu 10 Jun 2010 11:56:43 PM CEST
 LIBS:power
 LIBS:device
@@
 Sheet 3 6
 Title "sd2snes Mark II"
-Date "8 jun 2010"
+Date "10 jun 2010"
 Rev "A"
 Comp "Maximilian Rehkopf"
@@
 P 9500 5250
 F 0 "Q1" H 9500 5100 50  0000 R CNN
-F 1 "NPN" H 9500 5400 50  0000 R CNN
+F 1 "2N2222A" H 9500 5400 50  0000 R CNN
 	1    9500 5250
 	1    0    0    -1

Commit message: pcb wip
Parts:
- C15, C16, C17, R2, R3, R4: footprint (none) -> SM0805_FIXEDMASK
- D1, Q1: footprint (none) -> SOT23EBC
- U12: footprint (none) -> VFBGA54
- U13: footprint (none) -> VFBGA36
Changed lines of the file:
@@
-EESchema Schematic File Version 2  date Thu 10 Jun 2010 11:56:43 PM CEST
+EESchema Schematic File Version 2  date Fri 11 Jun 2010 11:43:50 PM CEST
 LIBS:power
 LIBS:device
@@
 Sheet 3 6
 Title "sd2snes Mark II"
-Date "10 jun 2010"
+Date "11 jun 2010"
 Rev "A"
 Comp "Maximilian Rehkopf"
@@
 Battery power OE switch
 $Comp
-L +3.3V #PWR109
+L +3.3V #PWR030
 U 1 1 4BF2FE97
 P 8350 5050
-F 0 "#PWR109" H 8350 5010 30  0001 C CNN
+F 0 "#PWR030" H 8350 5010 30  0001 C CNN
 F 1 "+3.3V" H 8350 5160 30  0000 C CNN
 	1    8350 5050
@@
 Connection ~ 9600 6050
 $Comp
-L GND #PWR111
+L GND #PWR031
 U 1 1 4BF2FE7B
 P 9600 6350
-F 0 "#PWR111" H 9600 6350 30  0001 C CNN
+F 0 "#PWR031" H 9600 6350 30  0001 C CNN
 F 1 "GND" H 9600 6280 30  0001 C CNN
 	1    9600 6350
@@
 F 0 "R4" V 9680 3600 50  0000 C CNN
 F 1 "20k" V 9600 3600 50  0000 C CNN
+F 2 "SM0805_FIXEDMASK" H 9600 3600 60  0001 C CNN
 	1    9600 3600
 	1    0    0    -1
@@
 F 0 "R3" V 9230 5700 50  0000 C CNN
 F 1 "1k" V 9150 5700 50  0000 C CNN
+F 2 "SM0805_FIXEDMASK" H 9150 5700 60  0001 C CNN
 	1    9150 5700
 	1    0    0    -1
@@
 F 0 "R2" V 8830 5250 50  0000 C CNN
 F 1 "4k7" V 8750 5250 50  0000 C CNN
+F 2 "SM0805_FIXEDMASK" H 8750 5250 60  0001 C CNN
 	1    8750 5250
 	0    1    1    0
@@
 F 0 "Q1" H 9500 5100 50  0000 R CNN
 F 1 "2N2222A" H 9500 5400 50  0000 R CNN
+F 2 "SOT23EBC" H 9500 5250 60  0001 C CNN
 	1    9500 5250
 	1    0    0    -1
 $EndComp
 $Comp
-L GND #PWR112
+L GND #PWR032
 U 1 1 4BF1A006
 P 10500 2000
-F 0 "#PWR112" H 10500 2000 30  0001 C CNN
+F 0 "#PWR032" H 10500 2000 30  0001 C CNN
 F 1 "GND" H 10500 1930 30  0001 C CNN
 	1    10500 2000
@@
 $EndComp
 $Comp
-L +BATT #PWR110
+L +BATT #PWR033
 U 1 1 4BF19EA4
 P 8400 1400
-F 0 "#PWR110" H 8400 1350 20  0001 C CNN
+F 0 "#PWR033" H 8400 1350 20  0001 C CNN
 F 1 "+BATT" H 8400 1500 30  0000 C CNN
 	1    8400 1400
@@
 $EndComp
 $Comp
-L +3.3V #PWR107
+L +3.3V #PWR034
 U 1 1 4BF19E7A
 P 6900 1400
-F 0 "#PWR107" H 6900 1360 30  0001 C CNN
+F 0 "#PWR034" H 6900 1360 30  0001 C CNN
 F 1 "+3.3V" H 6900 1510 30  0000 C CNN
 	1    6900 1400
@@
 F 0 "D1" H 7800 1475 60  0000 C CNN
 F 1 "BAT54C" H 7650 1750 60  0000 C CNN
+F 2 "SOT23EBC" H 7650 1600 60  0001 C CNN
 	1    7650 1600
 	1    0    0    -1
@@
 NoConn ~ 8500 4350
 $Comp
-L GND #PWR106
+L GND #PWR035
 U 1 1 4BCA30BF
 P 4750 5400
-F 0 "#PWR106" H 4750 5400 30  0001 C CNN
+F 0 "#PWR035" H 4750 5400 30  0001 C CNN
 F 1 "GND" H 4750 5330 30  0001 C CNN
 	1    4750 5400
@@
 F 0 "C17" H 3600 7100 50  0000 L CNN
 F 1 "100n" H 3600 6900 50  0000 L CNN
+F 2 "SM0805_FIXEDMASK" H 3550 7000 60  0001 C CNN
 	1    3550 7000
 	1    0    0    -1
@@
 F 0 "C16" H 10200 2100 50  0000 L CNN
 F 1 "100n" H 10200 1900 50  0000 L CNN
+F 2 "SM0805_FIXEDMASK" H 10150 2000 60  0001 C CNN
 	1    10150 2000
 	0    -1   1    0
@@
 F 0 "C15" H 3300 7100 50  0000 L CNN
 F 1 "100n" H 3300 6900 50  0000 L CNN
+F 2 "SM0805_FIXEDMASK" H 3250 7000 60  0001 C CNN
 	1    3250 7000
 	1    0    0    -1
 $EndComp
 $Comp
-L GND #PWR105
+L GND #PWR036
 U 1 1 4BAD3D2B
 P 3550 7300
-F 0 "#PWR105" H 3550 7300 30  0001 C CNN
+F 0 "#PWR036" H 3550 7300 30  0001 C CNN
 F 1 "GND" H 3550 7230 30  0001 C CNN
 	1    3550 7300
@@
 $EndComp
 $Comp
-L +1.8V #PWR104
+L +1.8V #PWR037
 U 1 1 4BAD3D27
 P 3550 6700
-F 0 "#PWR104" H 3550 6840 20  0001 C CNN
+F 0 "#PWR037" H 3550 6840 20  0001 C CNN
 F 1 "+1.8V" H 3550 6810 30  0000 C CNN
 	1    3550 6700
@@
 $EndComp
 $Comp
-L GND #PWR100
+L GND #PWR038
 U 1 1 4BAD3D20
 P 3250 7300
-F 0 "#PWR100" H 3250 7300 30  0001 C CNN
+F 0 "#PWR038" H 3250 7300 30  0001 C CNN
 F 1 "GND" H 3250 7230 30  0001 C CNN
 	1    3250 7300
@@
 $EndComp
 $Comp
-L +3.3V #PWR99
+L +3.3V #PWR039
 U 1 1 4BAD3D0B
 P 3250 6700
-F 0 "#PWR99" H 3250 6660 30  0001 C CNN
+F 0 "#PWR039" H 3250 6660 30  0001 C CNN
 F 1 "+3.3V" H 3250 6810 30  0000 C CNN
 	1    3250 6700
@@
 $EndComp
 $Comp
-L GND #PWR102
+L GND #PWR040
 U 1 1 4BAD33A7
 P 3400 5400
-F 0 "#PWR102" H 3400 5400 30  0001 C CNN
+F 0 "#PWR040" H 3400 5400 30  0001 C CNN
 F 1 "GND" H 3400 5330 30  0001 C CNN
 	1    3400 5400
@@
 $EndComp
 $Comp
-L GND #PWR108
+L GND #PWR041
 U 1 1 4BAD339F
 P 7650 5000
-F 0 "#PWR108" H 7650 5000 30  0001 C CNN
+F 0 "#PWR041" H 7650 5000 30  0001 C CNN
 F 1 "GND" H 7650 4930 30  0001 C CNN
 	1    7650 5000
@@
 $EndComp
 $Comp
-L +1.8V #PWR101
+L +1.8V #PWR042
 U 1 1 4BAD32D2
 P 3300 1550
-F 0 "#PWR101" H 3300 1690 20  0001 C CNN
+F 0 "#PWR042" H 3300 1690 20  0001 C CNN
 F 1 "+1.8V" H 3300 1660 30  0000 C CNN
 	1    3300 1550
@@
 $EndComp
 $Comp
-L +3.3V #PWR103
+L +3.3V #PWR043
 U 1 1 4BAD32BE
 P 3500 1550
-F 0 "#PWR103" H 3500 1510 30  0001 C CNN
+F 0 "#PWR043" H 3500 1510 30  0001 C CNN
 F 1 "+3.3V" H 3500 1660 30  0000 C CNN
 	1    3500 1550
@@
 F 0 "U13" H 7650 3550 60  0000 C CNN
 F 1 "CY62148EV30-BVXI" H 7700 3450 60  0000 C CNN
+F 2 "VFBGA36" H 7650 3450 60  0001 C CNN
 	1    7650 3450
 	1    0    0    -1
@@
 F 0 "U12" H 3400 3550 60  0000 C CNN
 F 1 "MT45W8MW16" H 3400 3450 60  0000 C CNN
+F 2 "VFBGA54" H 3400 3450 60  0001 C CNN
 	1    3400 3450
 	1    0    0    -1
